Commit message: feat(model): add foot contact sensor for cheater estimator
Note that foot force sensor's result has wrong orientation

File: dog_model/urdf/dog.xacro (robot description, xacro)
@@ -56,5 +56,5 @@
       name="${prefix}_foot">
       <xacro:dummy_inertial />
-      <collision>
+      <collision name="${prefix}_foot_collision">
         <origin
           xyz="0 0 0"

Commit message: feat(HalfFlipPlanner): change trajectory of the motion
Now, this planner can barely control the dog to do one flip.
The code is messy and needs to be refined.

File: dog_model/urdf/dog.xacro (robot description, xacro)
@@ -5,5 +5,5 @@
   <xacro:property name="PI" value="3.1415926535897931" />
   <xacro:property name="HIP_POS_X" value="0.23" />
-  <xacro:property name="HIP_POS_Y" value="0.0605" />
+  <xacro:property name="HIP_POS_Y" value="0.0805" />
   <xacro:property name="THIGH_POS_FROM_HIP_X" value="0.053" />
   <xacro:property name="THIGH_POS_FROM_HIP_Y" value="0.0575" />
@@ -167,5 +167,5 @@
   </link>
   <xacro:motor_joint joint="fr_hip_x" parent="fr_base" child="fr_hip"
-    lower="-1.60" upper="2.00">
+    lower="-1.60" upper="3.00">
     <origin xyz="0 0 0" rpy="0 0 0" />
     <axis xyz="-1 0 0" />
@@ -311,5 +311,5 @@
   </link>
   <xacro:motor_joint joint="fl_hip_x" parent="fl_base" child="fl_hip"
-    lower="-1.60" upper="2.00">
+    lower="-1.60" upper="3.00">
     <origin xyz="0 0 0" rpy="0 0 0" />
     <axis xyz="1 0 0" />
@@ -455,5 +455,5 @@
   </link>
   <xacro:motor_joint joint="bl_hip_x" parent="bl_base" child="bl_hip"
-    lower="-1.60" upper="2.00">
+    lower="-1.60" upper="3.00">
     <origin xyz="0 0 0" rpy="0 0 ${PI}" />
     <axis xyz="-1 0 0" />
@@ -599,5 +599,5 @@
   </link>
   <xacro:motor_joint joint="br_hip_x" parent="br_base" child="br_hip"
-    lower="-1.60" upper="2.00">
+    lower="-1.60" upper="3.00">
     <origin xyz="0 0 0" rpy="0 0 ${PI}" />
     <axis xyz="1 0 0" />

Commit message: feat(model): add an optional tail to the robot
The organization of the model file is also modified.

File: dog_model/urdf/dog.xacro (robot description, xacro)
@@ -1,696 +1,85 @@
 <?xml version="1.0" encoding="utf-8"?>
 <robot
-  name="dog"
-  xmlns:xacro="http://www.ros.org/wiki/xacro">
-  <xacro:property name="PI" value="3.1415926535897931" />
-  <xacro:property name="HIP_POS_X" value="0.23" />
-  <xacro:property name="HIP_POS_Y" value="0.0805" />
-  <xacro:property name="THIGH_POS_FROM_HIP_X" value="0.053" />
-  <xacro:property name="THIGH_POS_FROM_HIP_Y" value="0.0575" />
-  <xacro:property name="THIGH_LEN" value="0.2" />
-  <xacro:property name="SHIN_LEN" value="0.195" />
-  <xacro:property name="FOOT_RADIUS" value="0.0195" />
-  <xacro:include filename="$(find dog_model)/urdf/dog.gazebo" />
-  <xacro:macro name="dummy_inertial">
-    <inertial>
-      <origin
-        xyz="0 0 0"
-        rpy="0 0 0" />
-      <mass
-        value="1E-5" />
-      <inertia
-        ixx="1E-9"
-        ixy="0"
-        ixz="0"
-        iyy="1E-9"
-        iyz="0"
-        izz="1E-9" />
-    </inertial>
-  </xacro:macro>
-  <xacro:macro name="motor_joint"
-    params="joint *origin parent child *axis lower upper">
-    <joint
-      name="${joint}"
-      type="revolute">
-      <xacro:insert_block name="origin" />
-      <parent link="${parent}" />
-      <child link="${child}" />
-      <xacro:insert_block name="axis" />
-      <dynamics
-        damping="0.04"
-        friction="0.09" />
-      <limit
-        lower="${lower}"
-        upper="${upper}"
-        effort="17"
-        velocity="40" />
-      <safety_controller
-        soft_lower_limit="${lower + 0.01}"
-        soft_upper_limit="${upper - 0.01}"
-        k_velocity="100"
-        k_position="1000" />
-    </joint>
-  </xacro:macro>
-  <xacro:macro name="attach_foot" params="prefix">
-    <link
-      name="${prefix}_foot">
-      <xacro:dummy_inertial />
-      <collision name="${prefix}_foot_collision">
-        <origin
-          xyz="0 0 0"
-          rpy="0 0 0" />
-        <geometry>
-          <sphere
-            radius="${FOOT_RADIUS}" />
-        </geometry>
-      </collision>
-    </link>
-    <joint
-      name="${prefix}_fixed_foot"
-      type="fixed">
-      <origin
-        xyz="0 0 -${SHIN_LEN}"
-        rpy="0 0 0" />
-      <parent
-        link="${prefix}_shin" />
-      <child
-        link="${prefix}_foot" />
-    </joint>
-  </xacro:macro>
-  <link
-    name="torso">
-    <inertial>
-      <origin
-        xyz="0.000275 0 0.000266"
-        rpy="0 0 0" />
-      <mass
-        value="3.575" />
-      <inertia
-        ixx="0.017528444"
-        ixy="0"
-        ixz="0.000046175"
-        iyy="0.129944698"
-        iyz="0"
-        izz="0.143418825" />
-    </inertial>
-    <visual>
-      <origin
-        xyz="0 0 0"
-        rpy="0 0 0" />
-      <geometry>
-        <mesh
-          filename="package://dog_model/meshes/visualization/torso.stl" />
-      </geometry>
-      <material
-        name="">
-        <color
-          rgba="0.898039215686275 0.917647058823529 0.929411764705882 1" />
-      </material>
-    </visual>
-    <collision>
-      <origin
-        xyz="0 0 0"
-        rpy="0 0 0" />
-      <geometry>
-        <mesh
-          filename="package://dog_model/meshes/collision/torso.stl" />
-      </geometry>
-    </collision>
-  </link>
-  <link name="fr_base">
-    <xacro:dummy_inertial />
-  </link>
-  <joint name="fr_base_fixed" type="fixed">
-    <parent link="torso" />
-    <child link="fr_base" />
-    <origin xyz="${HIP_POS_X} -${HIP_POS_Y} 0" rpy="0 0 0" />
-  </joint>
-  <link
-    name="fr_hip">
-    <inertial>
-      <origin
-        xyz="0.050160 0.013329 1.2E-5"
-        rpy="0 0 0" />
-      <mass
-        value="0.650" />
-      <inertia
-        ixx="399.183E-6"
-        ixy="13.085E-6"
-        ixz="0.806E-6"
-        iyy="708.749E-6"
-        iyz="0.457E-6"
-        izz="460.327E-6" />
-    </inertial>
-    <visual>
-      <origin
-        xyz="0 0 0"
-        rpy="0 0 0" />
-      <geometry>
-        <mesh
-          filename="package://dog_model/meshes/visualization/fr_hip.stl" />
-      </geometry>
-      <material
-        name="">
-        <color
-          rgba="0.79216 0.81961 0.93333 1" />
-      </material>
-    </visual>
-    <collision>
-      <origin
-        xyz="0 0 0"
-        rpy="0 0 0" />
-      <geometry>
-        <mesh
-          filename="package://dog_model/meshes/collision/fr_hip.stl" />
-      </geometry>
-    </collision>
-  </link>
-  <xacro:motor_joint joint="fr_hip_x" parent="fr_base" child="fr_hip"
-    lower="-3.00" upper="3.00">
-    <origin xyz="0 0 0" rpy="0 0 0" />
-    <axis xyz="-1 0 0" />
-  </xacro:motor_joint>
-  <link
-    name="fr_thigh">
-    <inertial>
-      <origin
-        xyz="-0.019E-3 -29.693E-3 -13.531E-3"
-        rpy="0 0 0" />
-      <mass
-        value="0.863" />
-      <inertia
-        ixx="2082.653E-6"
-        ixy="0.090E-6"
-        ixz="-0.121E-6"
-        iyy="2271.664E-6"
-        iyz="261.229E-6"
-        izz="617.145E-6" />
-    </inertial>
-    <visual>
-      <origin
-        xyz="0 0 0"
-        rpy="0 0 0" />
-      <geometry>
-        <mesh
-          filename="package://dog_model/meshes/visualization/fr_thigh.stl" />
-      </geometry>
-      <material
-        name="">
-        <color
-          rgba="1 1 1 1" />
-      </material>
-    </visual>
-    <collision>
-      <origin
-        xyz="0 0 0"
-        rpy="0 0 0" />
-      <geometry>
-        <mesh
-          filename="package://dog_model/meshes/collision/thigh.stl" />
-      </geometry>
-    </collision>
-  </link>
-  <xacro:motor_joint joint="fr_hip_y" parent="fr_hip" child="fr_thigh"
-    lower="-3.89" upper="1.50">
-    <origin xyz="${THIGH_POS_FROM_HIP_X} -${THIGH_POS_FROM_HIP_Y} 0" rpy="0 0 0" />
-    <axis xyz="0 1 0" />
-  </xacro:motor_joint>
-  <link
-    name="fr_shin">
-    <inertial>
-      <origin
-        xyz="0 -0.012E-3 -93.811E-3"
-        rpy="0 0 0" />
-      <mass
-        value="0.119" />
-      <inertia
-        ixx="827.276E-6"
-        ixy="0"
-        ixz="0"
-        iyy="834.282E-6"
-        iyz="-0.116E-6"
-        izz="15.950E-6" />
-    </inertial>
-    <visual>
-      <origin
-        xyz="0 0 0"
-        rpy="0 0 ${PI}" />
-      <geometry>
-        <mesh
-          filename="package://dog_model/meshes/visualization/fl_shin.stl" />
-      </geometry>
-      <material
-        name="">
-        <color
-          rgba="0.89804 0.91765 0.92941 1" />
-      </material>
-    </visual>
-    <collision>
-      <origin
-        xyz="0 0 0"
-        rpy="0 0 0" />
-      <geometry>
-        <mesh
-          filename="package://dog_model/meshes/collision/shin.stl" />
-      </geometry>
-    </collision>
-  </link>
-  <xacro:motor_joint joint="fr_knee" parent="fr_thigh" child="fr_shin"
-    lower="-2.70" upper="2.70">
-    <origin xyz="0 0 -${THIGH_LEN}" rpy="0 0 0" />
-    <axis xyz="0 1 0" />
-  </xacro:motor_joint>
-  <xacro:attach_foot prefix="fr" />
-  <link name="fl_base">
-    <xacro:dummy_inertial />
-  </link>
-  <joint name="fl_base_fixed" type="fixed">
-    <parent link="torso" />
-    <child link="fl_base" />
-    <origin xyz="${HIP_POS_X} ${HIP_POS_Y} 0" rpy="0 0 0" />
-  </joint>
-  <link
-    name="fl_hip">
-    <inertial>
-      <origin
-        xyz="0.050160 -0.013329 1.2E-5"
-        rpy="0 0 0" />
-      <mass
-        value="0.650" />
-      <inertia
-        ixx="399.183E-6"
-        ixy="-13.085E-6"
-        ixz="0.806E-6"
-        iyy="708.749E-6"
-        iyz="-0.457E-6"
-        izz="460.327E-6" />
-    </inertial>
-    <visual>
-      <origin
-        xyz="0 0 0"
-        rpy="0 0 0" />
-      <geometry>
-        <mesh
-          filename="package://dog_model/meshes/visualization/fl_hip.stl" />
-      </geometry>
-      <material
-        name="">
-        <color
-          rgba="0.79216 0.81961 0.93333 1" />
-      </material>
-    </visual>
-    <collision>
-      <origin
-        xyz="0 0 0"
-        rpy="${PI} 0 0" />
-      <geometry>
-        <mesh
-          filename="package://dog_model/meshes/collision/fr_hip.stl" />
-      </geometry>
-    </collision>
-  </link>
-  <xacro:motor_joint joint="fl_hip_x" parent="fl_base" child="fl_hip"
-    lower="-3.00" upper="3.00">
-    <origin xyz="0 0 0" rpy="0 0 0" />
-    <axis xyz="1 0 0" />
-  </xacro:motor_joint>
-  <link
-    name="fl_thigh">
-    <inertial>
-      <origin
-        xyz="-0.019E-3 29.693E-3 -13.531E-3"
-        rpy="0 0 0" />
-      <mass
-        value="0.863" />
-      <inertia
-        ixx="2082.653E-6"
-        ixy="-0.090E-6"
-        ixz="-0.121E-6"
-        iyy="2271.664E-6"
-        iyz="-261.229E-6"
-        izz="617.145E-6" />
-    </inertial>
-    <visual>
-      <origin
-        xyz="0 0 0"
-        rpy="0 0 0" />
-      <geometry>
-        <mesh
-          filename="package://dog_model/meshes/visualization/fl_thigh.stl" />
-      </geometry>
-      <material
-        name="">
-        <color
-          rgba="1 1 1 1" />
-      </material>
-    </visual>
-    <collision>
-      <origin
-        xyz="0 0 0"
-        rpy="0 0 0" />
-      <geometry>
-        <mesh
-          filename="package://dog_model/meshes/collision/thigh.stl" />
-      </geometry>
-    </collision>
-  </link>
-  <xacro:motor_joint joint="fl_hip_y" parent="fl_hip" child="fl_thigh"
-    lower="-3.89" upper="1.50">
-    <origin xyz="${THIGH_POS_FROM_HIP_X} ${THIGH_POS_FROM_HIP_Y} 0" rpy="0 0 0" />
-    <axis xyz="0 1 0" />
-  </xacro:motor_joint>
-  <link
-    name="fl_shin">
-    <inertial>
-      <origin
-        xyz="0 0.012E-3 -93.811E-3"
-        rpy="0 0 0" />
-      <mass
-        value="0.119" />
-      <inertia
-        ixx="827.276E-6"
-        ixy="0"
-        ixz="0"
-        iyy="834.282E-6"
-        iyz="0.116E-6"
-        izz="15.950E-6" />
-    </inertial>
-    <visual>
-      <origin
-        xyz="0 0 0"
-        rpy="0 0 0" />
-      <geometry>
-        <mesh
-          filename="package://dog_model/meshes/visualization/fl_shin.stl" />
-      </geometry>
-      <material
-        name="">
-        <color
-          rgba="0.89804 0.91765 0.92941 1" />
-      </material>
-    </visual>
-    <collision>
-      <origin
-        xyz="0 0 0"
-        rpy="0 0 0" />
-      <geometry>
-        <mesh
-          filename="package://dog_model/meshes/collision/shin.stl" />
-      </geometry>
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