Commit message: feat(gazebo_pve_controller): enable simulation of mimic joints
The 'mimic joints' are a set of joints with mechianical connections,
which are constrained to perform same motions. The effort applied on
the joints are shared within the set in order to meet the constraint.

File: dog_model/urdf/tail.xacro (robot description, xacro)
@@ -3,4 +3,30 @@
     xmlns:xacro="http://www.ros.org/wiki/xacro">
     <xacro:macro name="attach_tail" params="parent_name">
+        <xacro:macro name="mimic_joint"
+            params="joint *origin parent child *axis lower upper use_friction">
+            <joint
+                name="${joint}"
+                type="revolute">
+                <xacro:insert_block name="origin" />
+                <parent link="${parent}" />
+                <child link="${child}" />
+                <xacro:insert_block name="axis" />
+                <xacro:if value="${use_friction}">
+                    <dynamics
+                        damping="${MOTOR_DAMPING}"
+                        friction="${MOTOR_FRICTION}" />
+                </xacro:if>
+                <limit
+                    lower="${lower}"
+                    upper="${upper}"
+                    effort="1000"
+                    velocity="${MOTOR_VELOCITY_MAX}" />
+                <safety_controller
+                    soft_lower_limit="${lower + 0.01}"
+                    soft_upper_limit="${upper - 0.01}"
+                    k_velocity="${MOTOR_TORQUE_KD}"
+                    k_position="${MOTOR_TORQUE_KP}" />
+            </joint>
+        </xacro:macro>
         <xacro:include filename="$(find dog_model)/urdf/defines.xacro" />
         <link name="tail_base">
@@ -81,5 +107,5 @@
         <xacro:motor_joint joint="tail_root_joint"
             parent="tail_base" child="tail_root"
-            lower="-3.00" upper="3.00">
+            lower="-3.14" upper="3.14">
             <origin xyz="${TAIL_POS_X} 0 ${TAIL_POS_Z}" rpy="0 0 0" />
             <axis xyz="0 0 1" />
@@ -122,10 +148,10 @@
             </collision>
         </link>
-        <xacro:motor_joint joint="tail_mid_joint"
+        <xacro:mimic_joint joint="tail_mid_joint"
             parent="tail_root" child="tail_mid"
-            lower="-3.00" upper="3.00">
+            lower="-2.00" upper="2.00" use_friction="false">
             <origin xyz="${- TAIL_ROOT_LEN} 0 0" rpy="0 0 0" />
             <axis xyz="0 1 0" />
-        </xacro:motor_joint>
+        </xacro:mimic_joint>
         <link name="tail_end">
             <inertial>
@@ -163,10 +189,10 @@
             </collision>
         </link>
-        <xacro:motor_joint joint="tail_end_joint"
+        <xacro:mimic_joint joint="tail_end_joint"
             parent="tail_mid" child="tail_end"
-            lower="-3.00" upper="3.00">
+            lower="-2.00" upper="2.00" use_friction="true">
             <origin xyz="${- TAIL_MID_LEN} 0 0" rpy="0 0 0" />
             <axis xyz="0 1 0" />
-        </xacro:motor_joint>
+        </xacro:mimic_joint>
     </xacro:macro>
 </robot>

Commit message: feat(model): add an optional weight for the tail
When the tail is applied, it may cause the CoM changes violently.
As a compensation, an optional weight can be attached to the torso
so the tail's weight can be partly balanced.

File: dog_model/urdf/tail.xacro (robot description, xacro)
@@ -2,4 +2,5 @@
 <robot
     xmlns:xacro="http://www.ros.org/wiki/xacro">
+    <xacro:arg name="add_tail_weight" default="false" />
     <xacro:macro name="attach_tail" params="parent_name">
         <xacro:macro name="mimic_joint"
@@ -195,4 +196,33 @@
             <axis xyz="0 1 0" />
         </xacro:mimic_joint>
+        <xacro:if value="$(arg add_tail_weight)" >
+            <link name="tail_weight">
+                <inertial>
+                    <origin
+                        xyz="0 0 0"
+                        rpy="0 0 0" />
+                    <mass
+                        value="2." />
+                    <inertia
+                        ixx="1E-9"
+                        ixy="0"
+                        ixz="0"
+                        iyy="1E-9"
+                        iyz="0"
+                        izz="1E-9" />
+                </inertial>
+            </link>
+            <joint
+                name="tail_weight_fixed"
+                type="fixed">
+                <origin
+                    xyz="0.1 0 0"
+                    rpy="0 0 0" />
+                <parent
+                    link="${parent_name}" />
+                <child
+                    link="tail_weight" />
+            </joint>
+        </xacro:if>
     </xacro:macro>
 </robot>
